File: schematics/src/ioboard/ioboard.brd (EAGLE design)
At the start: 99.1 x 35.6 mm, 18 parts

Commit message: Updated some schematics and docs
Parts:
- GLIDE, SIGN_ATTN: value ALPHA-9MMA -> 100k Lin
- RATE: value ALPHA-9MMA -> 1M log
Changed lines of the file:
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@@
 <?xml version="1.0" encoding="utf-8"?>
 <!DOCTYPE eagle SYSTEM "eagle.dtd">
-<eagle version="7.5.0">
+<eagle version="9.6.2">
 <drawing>
 <settings>
 <setting alwaysvectorfont="no"/>
+<setting keepoldvectorfont="yes"/>
 <setting verticaltext="up"/>
 </settings>
@@
 <param name="dpMaxLengthDifference" value="10mm"/>
 <param name="dpGapFactor" value="2.5"/>
-<param name="checkGrid" value="0"/>
 <param name="checkAngle" value="0"/>
 <param name="checkFont" value="1"/>
 <param name="checkRestrict" value="1"/>
+<param name="checkStop" value="0"/>
+<param name="checkValues" value="0"/>
+<param name="checkNames" value="1"/>
+<param name="checkWireStubs" value="1"/>
+<param name="checkPolygonWidth" value="0"/>
 <param name="useDiameter" value="13"/>
 <param name="maxErrors" value="50"/>
@@
 <attribute name="NAME" x="1.27" y="11.43" size="1.27" layer="21" font="vector"/>
 </element>
-<element name="SIGN_ATTN" library="TomW" package="EVUF" value="ALPHA-9MMA" x="20.955" y="26.67" smashed="yes" rot="R270">
+<element name="SIGN_ATTN" library="TomW" package="EVUF" value="100k Lin" x="20.955" y="26.67" smashed="yes" rot="R270">
 <attribute name="NAME" x="26.67" y="31.75" size="1.27" layer="25" font="vector" rot="R270"/>
 <attribute name="VALUE" x="17.145" y="30.48" size="1.27" layer="27" rot="R270"/>
 </element>
-<element name="RATE" library="TomW" package="EVUF" value="ALPHA-9MMA" x="57.785" y="26.67" smashed="yes" rot="R270">
+<element name="RATE" library="TomW" package="EVUF" value="1M log" x="57.785" y="26.67" smashed="yes" rot="R270">
 <attribute name="NAME" x="63.5" y="27.94" size="1.27" layer="25" font="vector" rot="R270"/>
 <attribute name="VALUE" x="53.975" y="30.48" size="1.27" layer="27" rot="R270"/>
@@
 <attribute name="VALUE" x="45.6946" y="19.5834" size="1.27" layer="27" ratio="10" rot="R180"/>
 </element>
-<element name="GLIDE" library="TomW" package="EVUF" value="ALPHA-9MMA" x="20.955" y="8.89" smashed="yes" rot="R270">
+<element name="GLIDE" library="TomW" package="EVUF" value="100k Lin" x="20.955" y="8.89" smashed="yes" rot="R270">
 <attribute name="NAME" x="26.67" y="12.7" size="1.27" layer="25" font="vector" rot="R270"/>
 <attribute name="VALUE" x="17.145" y="12.7" size="1.27" layer="27" rot="R270"/>
@@
 </signal>
 </signals>
+<mfgpreviewcolors>
+<mfgpreviewcolor name="soldermaskcolor" color="0xC8008000"/>
+<mfgpreviewcolor name="silkscreencolor" color="0xFFFEFEFE"/>
+<mfgpreviewcolor name="backgroundcolor" color="0xFF282828"/>
+<mfgpreviewcolor name="coppercolor" color="0xFFFFBF00"/>
+<mfgpreviewcolor name="substratecolor" color="0xFF786E46"/>
+</mfgpreviewcolors>
 </board>
 </drawing>
