File: schematics/src/ioboard/ioboard.sch (EAGLE design)
At the start: 18 parts

Commit message: Updated some schematics and docs
Parts:
- GLIDE, SIGN_ATTN: value ALPHA-9MMA -> 100k Lin
- RATE: value ALPHA-9MMA -> 1M log
Changed lines of the file:
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@@
 <part name="GND20" library="supply1" deviceset="GND" device=""/>
 <part name="GND21" library="supply1" deviceset="GND" device=""/>
-<part name="SIGN_ATTN" library="TomW" deviceset="ALPHA-9MM" device="A"/>
-<part name="RATE" library="TomW" deviceset="ALPHA-9MM" device="A"/>
+<part name="SIGN_ATTN" library="TomW" deviceset="ALPHA-9MM" device="A" value="100k Lin"/>
+<part name="RATE" library="TomW" deviceset="ALPHA-9MM" device="A" value="1M log"/>
 <part name="GND22" library="supply1" deviceset="GND" device=""/>
 <part name="GND23" library="supply1" deviceset="GND" device=""/>
@@
 <part name="LED1" library="led" deviceset="LED" device="3MM"/>
 <part name="GND38" library="supply1" deviceset="GND" device=""/>
-<part name="GLIDE" library="TomW" deviceset="ALPHA-9MM" device="A"/>
+<part name="GLIDE" library="TomW" deviceset="ALPHA-9MM" device="A" value="100k Lin"/>
 <part name="CLOCK_OUT" library="thonkiconn" deviceset="WQP-PJ301M-12_JACK" device="" value=""/>
 <part name="GND27" library="supply1" deviceset="GND" device=""/>
